File: cap_controller_hardware/upper/charger_JYC_RM2023_V1.2_control.kicad_pcb (KiCad board)
At the start: 4 copper layers, 83 x 58 mm, 235 parts, among them J1 Conn_02x02_Odd_Even, J10 Conn_02x02_Odd_Even, J11 Conn_01x03_MountingPin, J12 Conn_02x02_Odd_Even, J13 Conn_01x02_MountingPin, J2 Conn_02x02_Odd_Even, J3 Conn_02x03_Odd_Even, J4 Conn_02x02_Odd_Even, J5 Conn_01x04_MountingPin, J6 Conn_02x02_Odd_Even, J8 Conn_01x03_MountingPin, J9 Conn_01x04_MountingPin, Q1 AO3400A, U1 REF3033, U11 TJA1042T-3, U12 RS3236, U13 RS3236, U14 ISO_DC, U15 ISO_DC, U16 UCC27211D, U17 UCC27211D, U19 INA186, U2 STM32F334R8Tx, U3 RY8411, U4 RY8411, U5 GS8332-SR, U7 INA186, U8 INA186, U9 GS8332-SR, Y1 Crystal_GND2_Small

Commit message: Generating gerber and bom
Parts:
- C18: value 100nf -> 100n
- D1, D10, D11, D18, D2, D21, D8, D9: value D_Schottky -> K34
- D19, D20, D22: value D_TVS -> SMF10A
- D3: value D_TVS -> SMCJ28A; footprint Diode_SMD:D_SMC -> Diode_SMD:D_SMF
- J11, J8: value Conn_01x03_MountingPin -> Conn_UART
- J13: value Conn_01x02_MountingPin -> Conn_CAN
- J5: value Conn_01x04_MountingPin -> Conn_OLED
- J9: value Conn_01x04_MountingPin -> Conn_SWD
- L1, L2: value L -> 6R8
- Y1: value Crystal_GND2_Small -> 8MHz
