File: cap_controller_hardware/upper/charger_JYC_RM2023_V1.2_control.kicad_sch (KiCad schematic)
At the start: 176 parts, among them J1 Conn_02x02_Odd_Even, J10 Conn_02x02_Odd_Even, J11 Conn_UART, J12 Conn_02x02_Odd_Even, J13 Conn_CAN, J2 Conn_02x02_Odd_Even, J3 Conn_02x03_Odd_Even, J4 Conn_02x02_Odd_Even, J5 Conn_OLED, J6 Conn_02x02_Odd_Even, J8 Conn_UART, J9 Conn_SWD, Q1 AO3400A, U1 REF3033, U11 TJA1042T-3, U14 ISO_DC, U15 ISO_DC, U16 UCC27211D, U17 UCC27211D, U19 INA186, U2 STM32F334R8Tx, U5 GS8332-SR, U7 INA186, U8 INA186, U9 GS8332-SR, Y1 8MHz

Commit message: Generating gerber and bom
Parts:
- C18: value 100nf -> 100n
Changed lines of the file:
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@@
       (effects (font (size 1.27 1.27)) (justify left))
     )
-    (property "Value" "100nf" (at 181.356 148.59 0)
+    (property "Value" "100n" (at 181.356 148.59 0)
       (effects (font (size 1.27 1.27)) (justify left))
     )
